File: pcb/pcb.sch (KiCad schematic (older format))
At the start: 47 parts, among them J1 Conn_02x05_Odd_Even, J2 Conn_02x05_Odd_Even, J3 Conn_01x02, J4 Conn_01x06, J5 Conn_01x02, J6 Audio-Jack-3, J7 Conn_02x04_Top_Bottom, J8 Conn_01x04, J9 Conn_01x04, P1 Digital, P10 CONN_01X01, P11 CONN_01X01, P12 CONN_01X01, P13 CONN_01X01, P2 Power, P3 Analog, P4 Analog, P5 PWM, P6 PWM, P7 Communication, P8 CONN_01X01, P9 CONN_01X01, U1 POLOLU_A4988, U2 POLOLU_A4988, U3 L7809, U4 LTV-827

Commit message: updated schema files to match prototype pcb routing
Parts:
- gave numbers to parts that had none: 1
Changed lines of the file:
@@
 24
 Text Label 7000 1100 0    60   ~ 0
-25
+22
 Wire Wire Line
 	6750 2650 7100 2650
@@
 	6750 2750 7100 2750
 Text Label 6950 2750 0    60   ~ 0
+28
+Text Label 6950 2650 0    60   ~ 0
 26
-Text Label 6950 2650 0    60   ~ 0
-27
 Wire Wire Line
 	6750 2850 6750 2950
@@
 	1750 6900 2100 6900
 Text Label 1950 6900 0    60   ~ 0
-45
+49
 Wire Wire Line
 	1250 6700 950  6700
@@
 	1750 5800 2100 5800
 Text Label 1950 5800 0    60   ~ 0
-34
+46
 Wire Wire Line
 	1250 5800 950  5800
@@
 	1250 5700 950  5700
 Text Label 1000 5700 0    60   ~ 0
-43
+48
 $Comp
 L LTV-827 U4
@@
 shutter
 Text Label 5950 6500 0    60   ~ 0
-22
+32
 Text Label 5950 6800 0    60   ~ 0
-23
+30
 Text Notes 5750 650  0    60   ~ 0
 Motion/Stepper Control
@@
 	5400 4100 5400 5300
 $Comp
-L Conn_02x06_Odd_Even J?
+L Conn_02x06_Odd_Even J10
 U 1 1 59F6901C
 P 6150 4800
-F 0 "J?" H 6200 5100 50  0000 C CNN
+F 0 "J10" H 6200 5100 50  0000 C CNN
 F 1 "Conn_02x06_Odd_Even" H 6200 4400 50  0000 C CNN
 F 2 "" H 6150 4800 50  0001 C CNN
@@
 +5V
 $Comp
-L GND #PWR?
+L GND #PWR018
 U 1 1 59F69D09
 P 6800 5100
-F 0 "#PWR?" H 6800 4850 50  0001 C CNN
+F 0 "#PWR018" H 6800 4850 50  0001 C CNN
 F 1 "GND" H 6800 4950 50  0000 C CNN
 F 2 "" H 6800 5100 50  0001 C CNN
@@
 	6450 5000 6800 5000
 Text Label 6600 4600 0    60   ~ 0
-40
+34
 Text Label 6600 4700 0    60   ~ 0
-41
+35
 Text Label 6600 4800 0    60   ~ 0
-42
+36
 Text Label 6600 4900 0    60   ~ 0
-43
+37
 Text Label 6600 5000 0    60   ~ 0
-44
+38
 Text Notes 6050 4250 0    60   ~ 0
 I/O Aux
